File: hardware/boussole/boussole.kicad_pcb (KiCad board)
At the start: 2 copper layers, 0 parts

Commit message: PCB mechanical validation
Parts:
- added BT1: Battery, Battery:BatteryHolder_Keystone_3008_1x2450, B.Cu at (159.1, 118.4)
- added G***: LOGO, 0_stimulu-common:sinestimulus_logo, F.Cu at (151.6, 113.1)
- added J1: CX70M-24P1, 0_stimulu-common:USB-C_Female_CX70M-24P1, F.Cu at (167.6, 92.1)
- added REF**: NavSpark_SPU500F8, 0_stimulu-common:NavSpark_SPU500F8, F.Cu at (143.6, 96.1)
- added REF**: order_number, 0_stimulu-common:order_number, F.Cu at (152.9, 90.1)
- added REF**: SW_SPST_B3U-3000P-B, Button_Switch_SMD:SW_SPST_B3U-3000P-B, F.Cu at (143.5, 133.2)
- added REF**: SW_SPST_B3U-3000P-B, Button_Switch_SMD:SW_SPST_B3U-3000P-B, F.Cu at (155.7, 134.2)
- added REF**: SW_SPST_B3U-3000P-B, Button_Switch_SMD:SW_SPST_B3U-3000P-B, F.Cu at (167.1, 129.5)
- added REF**: SW_SPST_B3U-3000P-B, Button_Switch_SMD:SW_SPST_B3U-3000P-B, F.Cu at (175.1, 120.1)
- added REF**: SW_SPST_B3U-3000P-B, Button_Switch_SMD:SW_SPST_B3U-3000P-B, F.Cu at (178.0, 108.1)
- added REF**: MountingHole_2.2mm_M2_Pad, MountingHole:MountingHole_2.2mm_M2_Pad, F.Cu at (133.3, 126.5)
Routing:
- added copper zone on B.Cu, net Net-(J1-PadSH)
- added copper zone on F.Cu, net Net-(J1-PadSH)
Other:
- board outline added: 57.2 x 57.5 mm
- board text added: "190509 REV 1"
- board text added: "BOUSSOLE mechanical validation"
